Commit message: Update

File: robot_sim/urdf/robot.xacro (robot description, xacro)
@@ -5,11 +5,11 @@
   xmlns:xacro="http://ros.org/wiki/xacro"
   name="sick_tim">
-  <xacro:include filename="$(find robot_sim)/urdf/sick_tim.urdf.xacro" />
+  <xacro:include filename="$(find robot_sim_demo)/urdf/sick_tim.urdf.xacro" />
   <!-- Choose your laser -->
   <!--<xacro:sick_tim571 name="laser" ros_topic="scan"   />-->
   <xacro:rplidarA2 name="laser" ros_topic="scan"   />
-  <xacro:include filename="$(find robot_sim)/urdf/materials.xacro" />
-  <xacro:include filename="$(find robot_sim)/urdf/xbot-u.urdf.xacro" />
-  <xacro:include filename="$(find robot_sim)/urdf/xbot-u.gazebo" />
+  <xacro:include filename="$(find robot_sim_demo)/urdf/materials.xacro" />
+  <xacro:include filename="$(find robot_sim_demo)/urdf/xbot-u.urdf.xacro" />
+  <xacro:include filename="$(find robot_sim_demo)/urdf/xbot-u.gazebo" />
   <xacro:xbot2_base/>
 </robot>

File: robot_sim/urdf/sick_tim.urdf.xacro (robot description, xacro)
@@ -8,5 +8,5 @@
       length="0.06" width="0.06" height="0.079" mass="0.150" z_offset="0.05595"
       min_range="0.2" max_range="8.0"
-      mesh="package://robot_sim/models/meshes/rplidar.obj" />
+      mesh="package://robot_sim_demo/models/meshes/rplidar.dae" />
   </xacro:macro>
   <xacro:macro name="sick_tim310" params="name ros_topic">
@@ -14,5 +14,5 @@
       length="0.06" width="0.06" height="0.079" mass="0.150" z_offset="0.05595"
       min_range="0.05" max_range="4.0"
-      mesh="package://robot_sim/models/meshes/sick_tim310.stl" />
+      mesh="package://robot_sim_demo/models/meshes/sick_tim310.stl" />
   </xacro:macro>
   <xacro:macro name="sick_tim551" params="name ros_topic">
@@ -20,5 +20,5 @@
       length="0.06" width="0.06" height="0.086" mass="0.250" z_offset="0.06296"
       min_range="0.05" max_range="10.0"
-      mesh="package://robot_sim/models/meshes/sick_tim551.stl" />
+      mesh="package://robot_sim_demo/models/meshes/sick_tim551.stl" />
   </xacro:macro>
   <xacro:macro name="sick_tim571" params="name ros_topic">
@@ -26,5 +26,5 @@
       length="0.06" width="0.06" height="0.086" mass="0.250" z_offset="0.02"
       min_range="0.05" max_range="25.0"
-      mesh="package://robot_sim/models/meshes/sick_tim571.stl" />
+      mesh="package://robot_sim_demo/models/meshes/sick_tim571.stl" />
   </xacro:macro>
   <xacro:macro name="sick_tim" params="name ros_topic length width height mass z_offset min_range max_range mesh">
@@ -62,8 +62,8 @@
   </xacro:macro>
   <xacro:macro name="sick_tim_laser_gazebo_v0" params="name link ros_topic update_rate min_angle max_angle min_range max_range">
-    <!--gazebo reference="${link}">
+    <gazebo reference="${link}">
       <material value="Gazebo/LightWood" />
       <sensor type="gpu_ray" name="${name}">
-      <sensor type="ray" name="${name}">
+      <!--sensor type="ray" name="${name}"-->
         <always_on>true</always_on>
         <update_rate>${update_rate}</update_rate>
@@ -73,5 +73,5 @@
           <scan>
             <horizontal>
-              <samples>810</samples>
+              <samples>810</samples>  <!-- 810 -->
               <resolution>1</resolution>
               <min_angle>${min_angle}</min_angle>
@@ -86,5 +86,5 @@
         </ray>
         <plugin name="gazebo_ros_${name}_controller" filename="libgazebo_ros_gpu_laser.so">
-        <!plugin name="gazebo_ros_${name}_controller" filename="libgazebo_ros_laser.so" >
+        <!-- plugin name="gazebo_ros_${name}_controller" filename="libgazebo_ros_laser.so" -->
           <gaussianNoise>0.01</gaussianNoise>
           <alwaysOn>true</alwaysOn>
@@ -94,36 +94,5 @@
         </plugin>
       </sensor>
-    </gazebo-->
-  <gazebo reference="${link}">
-    <sensor type="ray" name="${name}">
-      <pose>0 0 0 0 0 0</pose>
-      <visualize>true</visualize>
-      <update_rate>20</update_rate>
-      <ray>
-        <scan>
-          <horizontal>
-            <samples>810</samples>
-            <resolution>1</resolution>
-            <min_angle>-1.570796</min_angle>
-            <max_angle>1.570796</max_angle>
-          </horizontal>
-        </scan>
-        <range>
-          <min>0.10</min>
-          <max>10.0</max>
-          <resolution>0.01</resolution>
-        </range>
-        <noise>
-          <type>gaussian</type>
-          <mean>0.0</mean>
-          <stddev>0.01</stddev>
-        </noise>
-      </ray>
-      <plugin name="gazebo_ros_head_hokuyo_controller" filename="libgazebo_ros_laser.so">
-        <topicName>${ros_topic}</topicName>
-        <frameName>${link}</frameName>
-      </plugin>
-    </sensor>
-  </gazebo>
+    </gazebo>
   </xacro:macro>
 </robot>

File: robot_sim/urdf/xbot-u.urdf.xacro (robot description, xacro)
@@ -21,5 +21,5 @@
       <origin xyz="0 0 0" rpy="0 0 0" />
       <geometry>
-        <mesh filename="package://robot_sim/models/meshes/base_link.obj" />
+        <mesh filename="package://robot_sim_demo/models/meshes/base_link.dae" />
       </geometry>
     </visual>
@@ -85,5 +85,5 @@
       <origin xyz="0 0 0" rpy="0 0 -1.57079632"/>
       <geometry>
-        <mesh filename="package://robot_sim/models/meshes/wheel.obj" />
+        <mesh filename="package://robot_sim_demo/models/meshes/wheel.dae" />
       </geometry>
     </visual>
@@ -112,5 +112,5 @@
       <origin xyz="0 0 0" rpy="0 0 1.57079632"/>
       <geometry>
-        <mesh filename="package://robot_sim/models/meshes/wheel.obj" />
+        <mesh filename="package://robot_sim_demo/models/meshes/wheel.dae" />
       </geometry>
     </visual>
@@ -138,5 +138,5 @@
       <origin xyz="0 0 0" rpy="0 0 1.57079632" />
       <geometry>
-        <mesh filename="package://robot_sim/models/meshes/yaw_platform.obj" />
+        <mesh filename="package://robot_sim_demo/models/meshes/yaw_platform.dae" />
       </geometry>
     </visual>
@@ -165,5 +165,5 @@
       <origin xyz="0 0 0" rpy="0 0 0" />
       <geometry>
-        <mesh filename="package://robot_sim/models/meshes/pitch_platform.obj" />
+        <mesh filename="package://robot_sim_demo/models/meshes/pitch_platform.dae" />
       </geometry>
     </visual>
@@ -195,5 +195,5 @@
       <geometry>
         <!--<mesh filename="package://robot_sim_demo/models/meshes/xtion_pro_camera.dae" />-->
-        <mesh filename="package://robot_sim/models/meshes/realsense.obj" />
+        <mesh filename="package://robot_sim_demo/models/meshes/realsense.dae" />
       </geometry>
     </visual>

Commit message: Update

File: robot_sim/urdf/robot.xacro (robot description, xacro)
@@ -5,11 +5,11 @@
   xmlns:xacro="http://ros.org/wiki/xacro"
   name="sick_tim">
-  <xacro:include filename="$(find robot_sim_demo)/urdf/sick_tim.urdf.xacro" />
+  <xacro:include filename="$(find robot_sim)/urdf/sick_tim.urdf.xacro" />
   <!-- Choose your laser -->
   <!--<xacro:sick_tim571 name="laser" ros_topic="scan"   />-->
   <xacro:rplidarA2 name="laser" ros_topic="scan"   />
-  <xacro:include filename="$(find robot_sim_demo)/urdf/materials.xacro" />
-  <xacro:include filename="$(find robot_sim_demo)/urdf/xbot-u.urdf.xacro" />
-  <xacro:include filename="$(find robot_sim_demo)/urdf/xbot-u.gazebo" />
+  <xacro:include filename="$(find robot_sim)/urdf/materials.xacro" />
+  <xacro:include filename="$(find robot_sim)/urdf/xbot-u.urdf.xacro" />
+  <xacro:include filename="$(find robot_sim)/urdf/xbot-u.gazebo" />
   <xacro:xbot2_base/>
 </robot>

File: robot_sim/urdf/sick_tim.urdf.xacro (robot description, xacro)
@@ -8,5 +8,5 @@
       length="0.06" width="0.06" height="0.079" mass="0.150" z_offset="0.05595"
       min_range="0.2" max_range="8.0"
-      mesh="package://robot_sim_demo/models/meshes/rplidar.dae" />
+      mesh="package://robot_sim/models/meshes/rplidar.dae" />
   </xacro:macro>
   <xacro:macro name="sick_tim310" params="name ros_topic">
@@ -14,5 +14,5 @@
       length="0.06" width="0.06" height="0.079" mass="0.150" z_offset="0.05595"
       min_range="0.05" max_range="4.0"
-      mesh="package://robot_sim_demo/models/meshes/sick_tim310.stl" />
+      mesh="package://robot_sim/models/meshes/sick_tim310.stl" />
   </xacro:macro>
   <xacro:macro name="sick_tim551" params="name ros_topic">
@@ -20,5 +20,5 @@
       length="0.06" width="0.06" height="0.086" mass="0.250" z_offset="0.06296"
       min_range="0.05" max_range="10.0"
-      mesh="package://robot_sim_demo/models/meshes/sick_tim551.stl" />
+      mesh="package://robot_sim/models/meshes/sick_tim551.stl" />
   </xacro:macro>
   <xacro:macro name="sick_tim571" params="name ros_topic">
@@ -26,5 +26,5 @@
       length="0.06" width="0.06" height="0.086" mass="0.250" z_offset="0.02"
       min_range="0.05" max_range="25.0"
-      mesh="package://robot_sim_demo/models/meshes/sick_tim571.stl" />
+      mesh="package://robot_sim/models/meshes/sick_tim571.stl" />
   </xacro:macro>
   <xacro:macro name="sick_tim" params="name ros_topic length width height mass z_offset min_range max_range mesh">

File: robot_sim/urdf/xbot-u.urdf.xacro (robot description, xacro)
@@ -21,5 +21,5 @@
       <origin xyz="0 0 0" rpy="0 0 0" />
       <geometry>
-        <mesh filename="package://robot_sim_demo/models/meshes/base_link.dae" />
+        <mesh filename="package://robot_sim/models/meshes/base_link.dae" />
       </geometry>
     </visual>
@@ -85,5 +85,5 @@
       <origin xyz="0 0 0" rpy="0 0 -1.57079632"/>
       <geometry>
-        <mesh filename="package://robot_sim_demo/models/meshes/wheel.dae" />
+        <mesh filename="package://robot_sim/models/meshes/wheel.dae" />
       </geometry>
     </visual>
@@ -112,5 +112,5 @@
       <origin xyz="0 0 0" rpy="0 0 1.57079632"/>
       <geometry>
-        <mesh filename="package://robot_sim_demo/models/meshes/wheel.dae" />
+        <mesh filename="package://robot_sim/models/meshes/wheel.dae" />
       </geometry>
     </visual>
@@ -138,5 +138,5 @@
       <origin xyz="0 0 0" rpy="0 0 1.57079632" />
       <geometry>
-        <mesh filename="package://robot_sim_demo/models/meshes/yaw_platform.dae" />
+        <mesh filename="package://robot_sim/models/meshes/yaw_platform.dae" />
       </geometry>
     </visual>
@@ -165,5 +165,5 @@
       <origin xyz="0 0 0" rpy="0 0 0" />
       <geometry>
-        <mesh filename="package://robot_sim_demo/models/meshes/pitch_platform.dae" />
+        <mesh filename="package://robot_sim/models/meshes/pitch_platform.dae" />
       </geometry>
     </visual>
@@ -194,6 +194,6 @@
       <origin xyz="0 0 0" rpy="0 0 0"/>
       <geometry>
-        <!--<mesh filename="package://robot_sim_demo/models/meshes/xtion_pro_camera.dae" />-->
-        <mesh filename="package://robot_sim_demo/models/meshes/realsense.dae" />
+        <!--<mesh filename="package://robot_sim/models/meshes/xtion_pro_camera.dae" />-->
+        <mesh filename="package://robot_sim/models/meshes/realsense.dae" />
       </geometry>
     </visual>
